Commit message: Test Tune PID

File: src/hexapod_description/robot/visual/hexapod.xacro (robot description, xacro)
@@ -5,4 +5,12 @@
     <xacro:include filename="$(find hexapod_description)/robot/visual/robot_material.xacro" />
     <xacro:include filename="$(find hexapod_description)/robot/visual/gazebo_full.xacro" />
+    <!-- WORLD LINK (for fixing base_link in space) -->
+    <link name="world"/>
+    <!-- FIXED JOINT: Lock base_link to world frame -->
+    <joint name="world_to_base" type="fixed">
+        <origin xyz="0 0 0.3" rpy="0 0 0" />  <!-- Fix base at 0.3m height -->
+        <parent link="world" />
+        <child link="base_link" />
+    </joint>
     <!-- BASE LINK -->
     <link name="base_link">

File: src/hexapod_description/robot/visual/hexapod_params.xacro (robot description, xacro)
@@ -26,15 +26,15 @@
     <xacro:property name="end_effector_joint_y" value="-0.00094278"/>
     <!-- JOINT LIMITS (radians) -->
-    <xacro:property name="joint_effort" value="10.0"/>
-    <xacro:property name="joint_velocity" value="5.0"/>
-    <!-- Hip joint limits -->
-    <xacro:property name="hip_lower_limit" value="-1.57"/>
-    <xacro:property name="hip_upper_limit" value="1.57"/>
-    <!-- Knee joint limits -->
-    <xacro:property name="knee_lower_limit" value="-2.0"/>
-    <xacro:property name="knee_upper_limit" value="2.0"/>
-    <!-- Ankle joint limits -->
-    <xacro:property name="ankle_lower_limit" value="-1.57"/>
-    <xacro:property name="ankle_upper_limit" value="1.57"/>
+    <xacro:property name="joint_effort" value="24.0"/>  <!-- Increased to 24 Nm -->
+    <xacro:property name="joint_velocity" value="10.0"/>  <!-- Increased to 10 rad/s -->
+    <!-- Hip joint limits: ±60° (120° total) to prevent collision with baselink -->
+    <xacro:property name="hip_lower_limit" value="-1.047"/>
+    <xacro:property name="hip_upper_limit" value="1.047"/>
+    <!-- Knee joint limits: ±45° (90° total) -->
+    <xacro:property name="knee_lower_limit" value="-0.785"/>
+    <xacro:property name="knee_upper_limit" value="0.785"/>
+    <!-- Ankle joint limits: ±45° (90° total) -->
+    <xacro:property name="ankle_lower_limit" value="-0.785"/>
+    <xacro:property name="ankle_upper_limit" value="0.785"/>
     <!-- JOINT DYNAMICS -->
     <!-- Hip joint -->
