Commit message: 001

File: src/hexapod_description/robot/visual/hexapod.urdf (robot description, URDF)
Before this commit: robot URDF_Full_Hexapod, 31 links, 30 joints
Links:
- added link foot_contact_1, mass 0.001; visual sphere radius=0.01
- added link foot_contact_2, mass 0.001; visual sphere radius=0.01
- added link foot_contact_3, mass 0.001; visual sphere radius=0.01
- added link foot_contact_4, mass 0.001; visual sphere radius=0.01
- added link foot_contact_5, mass 0.001; visual sphere radius=0.01
- added link foot_contact_6, mass 0.001; visual sphere radius=0.01
- added link world
- link ankle_link_1: geometry collision cylinder length=0.203 radius=0.038; visual mesh filename=package://hexapod_description/meshes/ankle_link_1.STL
- link ankle_link_2: geometry collision cylinder length=0.203 radius=0.038; visual mesh filename=package://hexapod_description/meshes/ankle_link_1.STL
- link ankle_link_3: geometry collision cylinder length=0.203 radius=0.038; visual mesh filename=package://hexapod_description/meshes/ankle_link_1.STL
- link ankle_link_4: geometry collision cylinder length=0.203 radius=0.038; visual mesh filename=package://hexapod_description/meshes/ankle_link_1.STL
- link ankle_link_5: geometry collision cylinder length=0.203 radius=0.038; visual mesh filename=package://hexapod_description/meshes/ankle_link_1.STL
- link ankle_link_6: geometry collision cylinder length=0.203 radius=0.038; visual mesh filename=package://hexapod_description/meshes/ankle_link_1.STL
- link base_link: geometry collision cylinder length=0.064 radius=0.11; visual mesh filename=package://hexapod_description/meshes/base_link.STL
- link end_effector_1: geometry collision box size=0.032 0.022 0.022; visual mesh filename=package://hexapod_description/meshes/end_effector_1.STL
- link end_effector_2: geometry collision box size=0.032 0.022 0.022; visual mesh filename=package://hexapod_description/meshes/end_effector_1.STL
- link end_effector_3: geometry collision box size=0.032 0.022 0.022; visual mesh filename=package://hexapod_description/meshes/end_effector_1.STL
- link end_effector_4: geometry collision box size=0.032 0.022 0.022; visual mesh filename=package://hexapod_description/meshes/end_effector_1.STL
- link end_effector_5: geometry collision box size=0.032 0.022 0.022; visual mesh filename=package://hexapod_description/meshes/end_effector_1.STL
- link end_effector_6: geometry collision box size=0.032 0.022 0.022; visual mesh filename=package://hexapod_description/meshes/end_effector_1.STL
- link foot_pointer_1: geometry collision box size=0.032 0.023 0.022; visual mesh filename=package://hexapod_description/meshes/foot_pointer_1.STL
- link foot_pointer_2: geometry collision box size=0.032 0.023 0.022; visual mesh filename=package://hexapod_description/meshes/foot_pointer_1.STL
- link foot_pointer_3: geometry collision box size=0.032 0.023 0.022; visual mesh filename=package://hexapod_description/meshes/foot_pointer_1.STL
- link foot_pointer_4: geometry collision box size=0.032 0.023 0.022; visual mesh filename=package://hexapod_description/meshes/foot_pointer_1.STL
- link foot_pointer_5: geometry collision box size=0.032 0.023 0.022; visual mesh filename=package://hexapod_description/meshes/foot_pointer_1.STL
- link foot_pointer_6: geometry collision box size=0.032 0.023 0.022; visual mesh filename=package://hexapod_description/meshes/foot_pointer_1.STL
- link hip_link_1: mass 0.111649772064324 -> 0.0882011859976947; geometry collision box size=0.126 0.061 0.077; visual mesh filename=package://hexapod_description/meshes/hip_link_1.STL
- link hip_link_2: geometry collision box size=0.126 0.061 0.077; visual mesh filename=package://hexapod_description/meshes/hip_link_1.STL
- link hip_link_3: mass 0.0882011859976946 -> 0.0882011859976947; geometry collision box size=0.126 0.061 0.077; visual mesh filename=package://hexapod_description/meshes/hip_link_1.STL
- link hip_link_4: geometry collision box size=0.126 0.061 0.077; visual mesh filename=package://hexapod_description/meshes/hip_link_1.STL
- link hip_link_5: geometry collision box size=0.126 0.061 0.077; visual mesh filename=package://hexapod_description/meshes/hip_link_1.STL
- link hip_link_6: mass 0.0882011859976949 -> 0.0882011859976947; geometry collision box size=0.126 0.061 0.077; visual mesh filename=package://hexapod_description/meshes/hip_link_1.STL
- link knee_link_1: geometry collision box size=0.134 0.129 0.080; visual mesh filename=package://hexapod_description/meshes/knee_link_1.STL
- link knee_link_2: geometry collision box size=0.134 0.129 0.080; visual mesh filename=package://hexapod_description/meshes/knee_link_1.STL
- link knee_link_3: geometry collision box size=0.134 0.129 0.080; visual mesh filename=package://hexapod_description/meshes/knee_link_1.STL
- link knee_link_4: geometry collision box size=0.134 0.129 0.080; visual mesh filename=package://hexapod_description/meshes/knee_link_1.STL
- link knee_link_5: geometry collision box size=0.134 0.129 0.080; visual mesh filename=package://hexapod_description/meshes/knee_link_1.STL
- link knee_link_6: geometry collision box size=0.134 0.129 0.080; visual mesh filename=package://hexapod_description/meshes/knee_link_1.STL
Joints:
- added joint foot_contact_joint_1: type fixed, parent end_effector_1, child foot_contact_1, origin xyz=-0.012 0.0015 0 rpy=0 0 0
- added joint foot_contact_joint_2: type fixed, parent end_effector_2, child foot_contact_2, origin xyz=-0.012 0.0015 0 rpy=0 0 0
- added joint foot_contact_joint_3: type fixed, parent end_effector_3, child foot_contact_3, origin xyz=-0.012 0.0015 0 rpy=0 0 0
- added joint foot_contact_joint_4: type fixed, parent end_effector_4, child foot_contact_4, origin xyz=-0.012 0.0015 0 rpy=0 0 0
- added joint foot_contact_joint_5: type fixed, parent end_effector_5, child foot_contact_5, origin xyz=-0.012 0.0015 0 rpy=0 0 0
- added joint foot_contact_joint_6: type fixed, parent end_effector_6, child foot_contact_6, origin xyz=-0.012 0.0015 0 rpy=0 0 0
- added joint world_to_base: type fixed, parent world, child base_link, origin xyz=0 0 0.5 rpy=0 0 0
- joint ankle_joint_1: limit lower=0 upper=0 effort=0 velocity=0 -> lower=-1.57 upper=1.57 effort=10.0 velocity=5.0
- joint ankle_joint_2: limit lower=0 upper=0 effort=0 velocity=0 -> lower=-1.57 upper=1.57 effort=10.0 velocity=5.0
- joint ankle_joint_3: limit lower=0 upper=0 effort=0 velocity=0 -> lower=-1.57 upper=1.57 effort=10.0 velocity=5.0
- joint ankle_joint_4: limit lower=0 upper=0 effort=0 velocity=0 -> lower=-1.57 upper=1.57 effort=10.0 velocity=5.0
- joint ankle_joint_5: limit lower=0 upper=0 effort=0 velocity=0 -> lower=-1.57 upper=1.57 effort=10.0 velocity=5.0
- joint ankle_joint_6: limit lower=0 upper=0 effort=0 velocity=0 -> lower=-1.57 upper=1.57 effort=10.0 velocity=5.0
- joint end_effector_joint_1: axis 0 0 0 -> (none)
- joint end_effector_joint_2: axis 0 0 0 -> (none)
- joint end_effector_joint_3: axis 0 0 0 -> (none)
- joint end_effector_joint_4: axis 0 0 0 -> (none)
- joint end_effector_joint_5: axis 0 0 0 -> (none)
- joint end_effector_joint_6: axis 0 0 0 -> (none)
- joint foot_pointer_joint_1: axis 0 0 0 -> (none)
- joint foot_pointer_joint_2: axis 0 0 0 -> (none)
- joint foot_pointer_joint_3: axis 0 0 0 -> (none)
- joint foot_pointer_joint_4: axis 0 0 0 -> (none)
- joint foot_pointer_joint_5: axis 0 0 0 -> (none)
- joint foot_pointer_joint_6: axis 0 0 0 -> (none)
- joint hip_joint_1: limit lower=0 upper=0 effort=0 velocity=0 -> lower=-1.57 upper=1.57 effort=10.0 velocity=5.0
- joint hip_joint_2: limit lower=0 upper=0 effort=0 velocity=0 -> lower=-1.57 upper=1.57 effort=10.0 velocity=5.0
- joint hip_joint_3: limit lower=0 upper=0 effort=0 velocity=0 -> lower=-1.57 upper=1.57 effort=10.0 velocity=5.0
- joint hip_joint_4: limit lower=0 upper=0 effort=0 velocity=0 -> lower=-1.57 upper=1.57 effort=10.0 velocity=5.0
- joint hip_joint_5: limit lower=0 upper=0 effort=0 velocity=0 -> lower=-1.57 upper=1.57 effort=10.0 velocity=5.0
- joint hip_joint_6: limit lower=0 upper=0 effort=0 velocity=0 -> lower=-1.57 upper=1.57 effort=10.0 velocity=5.0
- joint knee_joint_1: limit lower=0 upper=0 effort=0 velocity=0 -> lower=-2.0 upper=2.0 effort=10.0 velocity=5.0
- joint knee_joint_2: limit lower=0 upper=0 effort=0 velocity=0 -> lower=-2.0 upper=2.0 effort=10.0 velocity=5.0
- joint knee_joint_3: limit lower=0 upper=0 effort=0 velocity=0 -> lower=-2.0 upper=2.0 effort=10.0 velocity=5.0
- joint knee_joint_4: limit lower=0 upper=0 effort=0 velocity=0 -> lower=-2.0 upper=2.0 effort=10.0 velocity=5.0
- joint knee_joint_5: limit lower=0 upper=0 effort=0 velocity=0 -> lower=-2.0 upper=2.0 effort=10.0 velocity=5.0
- joint knee_joint_6: limit lower=0 upper=0 effort=0 velocity=0 -> lower=-2.0 upper=2.0 effort=10.0 velocity=5.0
